Commit message: feat: add fleet base station and cooperative simulation

File: src/uav_usv_sim/urdf/landing_boat.urdf.xacro (robot description, xacro)
@@ -5,5 +5,5 @@
       <origin xyz="0 0 0" rpy="0 0 0"/>
       <geometry>
-        <box size="3.4 1.9 0.5"/>
+        <box size="5.61 3.135 0.625"/>
       </geometry>
       <material name="boat_black">
@@ -16,5 +16,5 @@
     <parent link="base_link"/>
     <child link="hull/front_lidar"/>
-    <origin xyz="0.55 0 1.55" rpy="0 0 0"/>
+    <origin xyz="0.9075 0 1.5625" rpy="0 0 0"/>
   </joint>
   <link name="mid360_link"/>
@@ -22,5 +22,5 @@
     <parent link="base_link"/>
     <child link="mid360_link"/>
-    <origin xyz="0.55 0 1.55" rpy="0 0 0"/>
+    <origin xyz="0.9075 0 1.5625" rpy="0 0 0"/>
   </joint>
   <link name="front_camera_link"/>
@@ -28,5 +28,5 @@
     <parent link="base_link"/>
     <child link="front_camera_link"/>
-    <origin xyz="1.405 0 0.86" rpy="0 0 0"/>
+    <origin xyz="2.31825 0 1.075" rpy="0 0 0"/>
   </joint>
   <link name="imu_link"/>
@@ -34,5 +34,5 @@
     <parent link="base_link"/>
     <child link="imu_link"/>
-    <origin xyz="0 0 0.45" rpy="0 0 0"/>
+    <origin xyz="0 0 0.5625" rpy="0 0 0"/>
   </joint>
   <link name="landing_pad_link"/>
@@ -40,5 +40,5 @@
     <parent link="base_link"/>
     <child link="landing_pad_link"/>
-    <origin xyz="-0.92 0 0.43" rpy="0 0 0"/>
+    <origin xyz="-1.518 0 0.56" rpy="0 0 0"/>
   </joint>
 </robot>
